File: hardware/jank.kicad_pcb (KiCad board)
At the start: 2 copper layers, 80 x 127.5 mm, 69 parts, among them J1 usb-c, J2 AVR-ISP, M0 KEY_LED, M1 KEY_LED, M2 KEY_LED, M3 KEY_LED, SW0 SW_Push, U1 ATmega32U4-AU, U2 MP3202, Y1 16MHz

Commit message: Renaming project and repo from numpty to jank.
Parts:
- D1: value Schottky -> 30V_500mA_Schottky
- G*** (x2): footprint numpty:osha_logo_8mm -> jank:osha_logo_8mm
- G*** (x2): footprint numpty:clewsy_logo_8mm -> jank:clewsy_logo_8mm
- L1: footprint numpty:SRN3010TA -> jank:SRN3010TA
- SW_0: renamed from 0; footprint numpty:Gateron_LED_1.00u_Plate -> jank:Gateron_LED_1.00u_Plate
- SW_1: renamed from 1; footprint numpty:Gateron_LED_1.00u_Plate -> jank:Gateron_LED_1.00u_Plate
- SW_2: renamed from 2; footprint numpty:Gateron_LED_1.00u_Plate -> jank:Gateron_LED_1.00u_Plate
- SW_3: renamed from 3; footprint numpty:Gateron_LED_1.00u_Plate -> jank:Gateron_LED_1.00u_Plate
- SW_4: renamed from 4; footprint numpty:Gateron_LED_1.00u_Plate -> jank:Gateron_LED_1.00u_Plate
- SW_5: renamed from 5; footprint numpty:Gateron_LED_1.00u_Plate -> jank:Gateron_LED_1.00u_Plate
- SW_6: renamed from 6; footprint numpty:Gateron_LED_1.00u_Plate -> jank:Gateron_LED_1.00u_Plate
- SW_7: renamed from 7; footprint numpty:Gateron_LED_1.00u_Plate -> jank:Gateron_LED_1.00u_Plate
- SW_8: renamed from 8; footprint numpty:Gateron_LED_1.00u_Plate -> jank:Gateron_LED_1.00u_Plate
- SW_9: renamed from 9; footprint numpty:Gateron_LED_1.00u_Plate -> jank:Gateron_LED_1.00u_Plate
- SW_DIV0: renamed from /; footprint numpty:Gateron_LED_1.00u_Plate -> jank:Gateron_LED_1.00u_Plate
- SW_ENT0: renamed from ENTER; footprint numpty:Gateron_LED_1.00u_Plate -> jank:Gateron_LED_1.00u_Plate
- SW_M0: renamed from M0; footprint numpty:Gateron_LED_1.00u_Plate -> jank:Gateron_LED_1.00u_Plate
- SW_M1: renamed from M1; footprint numpty:Gateron_LED_1.00u_Plate -> jank:Gateron_LED_1.00u_Plate
- SW_M2: renamed from M2; footprint numpty:Gateron_LED_1.00u_Plate -> jank:Gateron_LED_1.00u_Plate
- SW_M3: renamed from M3; footprint numpty:Gateron_LED_1.00u_Plate -> jank:Gateron_LED_1.00u_Plate
- SW_MIN0: renamed from -; footprint numpty:Gateron_LED_1.00u_Plate -> jank:Gateron_LED_1.00u_Plate
- SW_MUL0: renamed from *; footprint numpty:Gateron_LED_1.00u_Plate -> jank:Gateron_LED_1.00u_Plate
- SW_NL0: renamed from NUMLOCK; footprint numpty:Gateron_LED_1.00u_Plate -> jank:Gateron_LED_1.00u_Plate
- SW_PER0: renamed from .; footprint numpty:Gateron_LED_1.00u_Plate -> jank:Gateron_LED_1.00u_Plate
- SW_PLU0: renamed from +; footprint numpty:Gateron_LED_1.00u_Plate -> jank:Gateron_LED_1.00u_Plate
- U2: footprint Package_TO_SOT_SMD:TSOT-23-6_HandSoldering -> Package_TO_SOT_SMD:SOT-23-6_Handsoldering
Routing:
- net LEDS_ANODE: track 139.9 -> 140.5 mm
